File: QuadPinDriver/QuadPinDriver.sch (KiCad schematic (older format))
At the start: 22 parts

Commit message: Octal -> Quad
Parts:
- removed C? (x5): 100n, symbol Device:C_Small
- removed C? (x3): 1u, symbol Device:CP_Small
- removed U? (x5): 74HC00, symbol 74xx:74HC00
- removed U?: DAC7614U, Package_SO:SOIC-16W_7.5x10.3mm_P1.27mm, symbol UniProg:DAC7614U
Connections:
- net labels removed: DAC4, DAC5, DAC6, DAC7, D_SEL, M_DATA, PIN4, PIN5, PIN6, PIN7, ~D_SEL
- wire segments 153 -> 86
- no-connect marks 3 -> 0
